File: ActiveHPF/ActiveHPF.sch (KiCad schematic (older format))
At the start: 16 parts

Commit message: Added annotations
Parts:
- gave numbers to parts that had none: 14
Changed lines of the file:
@@
 $EndDescr
 $Comp
-L Amplifier_Operational:TL072 U?
+L Amplifier_Operational:TL072 U1
 U 1 1 60DA7AB5
 P 4400 3950
-F 0 "U?" H 4475 4200 50  0000 C CNN
+F 0 "U1" H 4475 4200 50  0000 C CNN
 F 1 "TL072" H 4475 4125 50  0000 C CNN
 F 2 "" H 4400 3950 50  0001 C CNN
@@
 $EndComp
 $Comp
-L Amplifier_Operational:TL072 U?
+L Amplifier_Operational:TL072 U1
 U 2 1 60DA8706
 P 6150 4050
-F 0 "U?" H 6250 4300 50  0000 C CNN
+F 0 "U1" H 6250 4300 50  0000 C CNN
 F 1 "TL072" H 6250 4225 50  0000 C CNN
 F 2 "" H 6150 4050 50  0001 C CNN
@@
 $EndComp
 $Comp
-L Amplifier_Operational:TL072 U?
+L Amplifier_Operational:TL072 U1
 U 3 1 60DA9AD0
 P 6150 4050
-F 0 "U?" H 6108 4050 50  0001 L CNN
+F 0 "U1" H 6108 4050 50  0001 L CNN
 F 1 "TL072" H 6108 4005 50  0001 L CNN
 F 2 "" H 6150 4050 50  0001 C CNN
@@
 $EndComp
 $Comp
-L power:+12V #PWR?
+L power:+12V #PWR06
 U 1 1 60DB38AA
 P 6050 3725
-F 0 "#PWR?" H 6050 3575 50  0001 C CNN
+F 0 "#PWR06" H 6050 3575 50  0001 C CNN
 F 1 "+12V" H 6065 3898 50  0000 C CNN
 F 2 "" H 6050 3725 50  0001 C CNN
@@
 $EndComp
 $Comp
-L power:-12V #PWR?
+L power:-12V #PWR07
 U 1 1 60DB44BC
 P 6050 4400
-F 0 "#PWR?" H 6050 4500 50  0001 C CNN
+F 0 "#PWR07" H 6050 4500 50  0001 C CNN
 F 1 "-12V" H 6065 4573 50  0000 C CNN
 F 2 "" H 6050 4400 50  0001 C CNN
@@
 	6050 4350 6050 4400
 $Comp
-L Device:R R?
+L Device:R R3
 U 1 1 60DEAD4C
 P 5575 3950
-F 0 "R?" V 5500 3950 50  0000 C CNN
+F 0 "R3" V 5500 3950 50  0000 C CNN
 F 1 "560" V 5575 3950 50  0000 C CNN
 F 2 "" V 5505 3950 50  0001 C CNN
@@
 	5725 3950 5850 3950
 $Comp
-L Device:C C?
+L Device:C C1
 U 1 1 60E16F41
 P 5000 3950
-F 0 "C?" V 4800 3950 50  0000 C CNN
+F 0 "C1" V 4800 3950 50  0000 C CNN
 F 1 "10nF" V 4875 3950 50  0000 C CNN
 F 2 "" H 5038 3800 50  0001 C CNN
@@
 $EndComp
 $Comp
-L power:GND #PWR?
+L power:GND #PWR03
 U 1 1 60DF3B50
 P 5100 3350
-F 0 "#PWR?" H 5100 3100 50  0001 C CNN
+F 0 "#PWR03" H 5100 3100 50  0001 C CNN
 F 1 "GND" H 5105 3177 50  0000 C CNN
 F 2 "" H 5100 3350 50  0001 C CNN
@@
 	5300 2575 5375 2575
 $Comp
-L Device:LED D?
+L Device:LED D1
 U 1 1 60DD7F41
 P 5525 2575
-F 0 "D?" H 5518 2320 50  0000 C CNN
+F 0 "D1" H 5518 2320 50  0000 C CNN
 F 1 "LED" H 5518 2411 50  0000 C CNN
 F 2 "" H 5525 2575 50  0001 C CNN
@@
 	5300 2675 5300 2575
 $Comp
-L Isolator:VTL5C U?
+L Isolator:VTL5C U2
 U 1 1 60DCC12E
 P 5200 2975
-F 0 "U?" V 5150 2525 50  0000 L CNN
+F 0 "U2" V 5150 2525 50  0000 L CNN
 F 1 "DIY Vactrol" V 5225 2375 50  0000 L CNN
 F 2 "OptoDevice:PerkinElmer_VTL5C" H 5200 2975 50  0001 C CNN
@@
 	6550 4050 6450 4050
 $Comp
-L Device:R R?
+L Device:R R5
 U 1 1 60E4EFD6
 P 6075 4800
-F 0 "R?" V 6000 4800 50  0000 C CNN
+F 0 "R5" V 6000 4800 50  0000 C CNN
 F 1 "10k" V 6075 4800 50  0000 C CNN
 F 2 "" V 6005 4800 50  0001 C CNN
@@
 $EndComp
 $Comp
-L Device:R R?
+L Device:R R4
 U 1 1 60E50BF6
 P 5750 5075
-F 0 "R?" H 5650 5075 50  0000 C CNN
+F 0 "R4" H 5650 5075 50  0000 C CNN
 F 1 "20k" V 5750 5075 50  0000 C CNN
 F 2 "" V 5680 5075 50  0001 C CNN
@@
 	6550 4050 6550 4800
 $Comp
-L power:GND #PWR?
+L power:GND #PWR05
 U 1 1 60E5533B
 P 5750 5375
-F 0 "#PWR?" H 5750 5125 50  0001 C CNN
+F 0 "#PWR05" H 5750 5125 50  0001 C CNN
 F 1 "GND" H 5755 5202 50  0000 C CNN
 F 2 "" H 5750 5375 50  0001 C CNN
@@
 	5750 5225 5750 5375
 $Comp
-L Device:R R?
+L Device:R R6
 U 1 1 60E593B8
 P 6800 4050
-F 0 "R?" V 6725 4050 50  0000 C CNN
+F 0 "R6" V 6725 4050 50  0000 C CNN
 F 1 "1k" V 6800 4050 50  0000 C CNN
 F 2 "" V 6730 4050 50  0001 C CNN
@@
 Connection ~ 6550 4050
 $Comp
-L Device:R R?
+L Device:R R1
 U 1 1 60E66E66
 P 4625 2400
-F 0 "R?" V 4550 2400 50  0000 C CNN
+F 0 "R1" V 4550 2400 50  0000 C CNN
 F 1 "1k" V 4625 2400 50  0000 C CNN
 F 2 "" V 4555 2400 50  0001 C CNN
@@
 $EndComp
 $Comp
-L Device:R R?
+L Device:R R2
 U 1 1 60E67584
 P 4625 2625
-F 0 "R?" V 4550 2625 50  0000 C CNN
+F 0 "R2" V 4550 2625 50  0000 C CNN
 F 1 "1k" V 4625 2625 50  0000 C CNN
 F 2 "" V 4555 2625 50  0001 C CNN
@@
 	5100 2625 5100 2675
 $Comp
-L Connector:TestPoint TP?
+L Connector:TestPoint TP2
 U 1 1 60E77D06
 P 4275 2400
-F 0 "TP?" V 4470 2472 50  0000 C CNN
+F 0 "TP2" V 4470 2472 50  0000 C CNN
 F 1 "CV_IN" V 4379 2472 50  0000 C CNN
 F 2 "" H 4475 2400 50  0001 C CNN
@@
 	4275 2400 4475 2400
 $Comp
-L Connector:TestPoint TP?
+L Connector:TestPoint TP1
 U 1 1 60E829D6
 P 3875 3850
-F 0 "TP?" V 4070 3922 50  0000 C CNN
+F 0 "TP1" V 4070 3922 50  0000 C CNN
 F 1 "AUDIO_IN" V 3979 3922 50  0000 C CNN
 F 2 "" H 4075 3850 50  0001 C CNN
@@
 $EndComp
 $Comp
-L Connector:TestPoint TP?
+L Connector:TestPoint TP3
 U 1 1 60E842B1
 P 7150 4050
-F 0 "TP?" V 7104 4238 50  0000 L CNN
+F 0 "TP3" V 7104 4238 50  0000 L CNN
 F 1 "AUDIO_OUT" V 7195 4238 50  0000 L CNN
 F 2 "" H 7350 4050 50  0001 C CNN
@@
 	3875 3850 4100 3850
 $Comp
-L power:GND #PWR?
+L power:GND #PWR04
 U 1 1 60DD5AD0
 P 5750 2750
-F 0 "#PWR?" H 5750 2500 50  0001 C CNN
+F 0 "#PWR04" H 5750 2500 50  0001 C CNN
 F 1 "GND" H 5755 2577 50  0000 C CNN
 F 2 "" H 5750 2750 50  0001 C CNN
@@
 	5750 2575 5750 2750
 $Comp
-L Device:R_POT RV?
+L Device:R_POT RV1
 U 1 1 60EA15D8
 P 3725 2625
-F 0 "RV?" H 3655 2671 50  0000 R CNN
+F 0 "RV1" H 3655 2671 50  0000 R CNN
 F 1 "CV_OFFSET" H 3655 2580 50  0000 R CNN
 F 2 "" H 3725 2625 50  0001 C CNN
@@
 	3875 2625 4475 2625
 $Comp
-L power:+12V #PWR?
+L power:+12V #PWR01
 U 1 1 60EA3C91
 P 3725 2325
-F 0 "#PWR?" H 3725 2175 50  0001 C CNN
+F 0 "#PWR01" H 3725 2175 50  0001 C CNN
 F 1 "+12V" H 3740 2498 50  0000 C CNN
 F 2 "" H 3725 2325 50  0001 C CNN
@@
 $EndComp
 $Comp
-L power:GND #PWR?
+L power:GND #PWR02
 U 1 1 60EA4530
 P 3725 2925
-F 0 "#PWR?" H 3725 2675 50  0001 C CNN
+F 0 "#PWR02" H 3725 2675 50  0001 C CNN
 F 1 "GND" H 3730 2752 50  0000 C CNN
 F 2 "" H 3725 2925 50  0001 C CNN
